File: Moyka_E4.kicad_sch (KiCad schematic)
At the start: 1 part, among them J1 DE9_Plug

Commit message: VER1: исправил ошибки
Other:
- note added: "X1"
- note added: "X10"
- note added: "X2"
- note added: "X3"
- note added: "X4"
- note added: "X5"
- note added: "X6"
- note added: "X7"
- note added: "X8"
- note added: "X9"

Commit message: VER1: добавил нумерацию проводов и убрал УГО
Parts:
- removed J1: DE9_Plug, symbol Connector:DE9_Plug
Other:
- note added: "X11"
- note added: "К единой электроэнергетической системе"
- note removed: "M"
- note removed: "t°"

Commit message: VER1: добавил децимальники жгутов
Other:
- note added: "A1-X1"
- note added: "A1-X2"
- note added: "A1-X3"
- note added: "A1-X4"
- note added: "A10-X1"
- note added: "A11-X1"
- note added: "A2-X1"
- note added: "A2-X10"
- note added: "A2-X11"
- note added: "A2-X2"
- note added: "A2-X3"
- note added: "A2-X4"
- note added: "A2-X5"
- note added: "A2-X6"
- note added: "A2-X7"
- note added: "A2-X8"
- note added: "A2-X9"
- note added: "A3-X1"
- note added: "A4-X1"
- note added: "A4-X2"
- note added: "A6-X1"
- note added: "A7-X1"
- note added: "A8-X1"
- note added: "A9-X1"
- note added: "CAN разъём"
- note added: "XT1"
- note added: "XT2"
- note added: "А1"
- note added: "А10"
- note added: "А11"
- note added: "А2"
- note added: "А3"
- note added: "А4"
- note added: "А5"
- note added: "А6"
- note added: "А7"
- note added: "А8"
- note added: "А9"
- title: (none) -> Схема электрическая соединений

Commit message: VER1: добавил в таблицу кабели
Other:
- company: (none) -> ООО "Электротранспортные технологии"

Commit message: VER1: скинул на проверку Лёше
Other:
- note added: "НВЦТ.0001.0000.100"
- note removed: "A10-X1"
- note removed: "А11"
