File: Moyka_E4.kicad_sch (KiCad schematic)
At the start: 0 parts

Commit message: VER1: начал переделывать таблицу
Other:
- note removed: "A11-X1"

Commit message: VER1: почти закончил таблицу
Other:
- note added: "A2-X12"
- note added: "A2-X13"
- note added: "X12"
- note added: "X13"
- note added: "Питание 24В аварийное"
- note added: "Питание 24В штатное"

Commit message: VER1: закончил таблицу
Other:
- note added: "ООО "Электротранспортные"
- note added: "Схема электрическая соединений"
- note added: "технологии""
- company: ООО "Электротранспортные технологии" -> (none)
- title: Схема электрическая соединений -> Система электродвижения

Commit message: VER1: исправил децимальник
Other:
- note removed: "НВЦТ.0001.0000.100"
Changed lines of the file:
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@@
 		(title "Система электродвижения")
 		(date "2025-04-15")
-		(comment 1 "НВЦТ.0001.0000.100 Э4")
+		(comment 1 "650232.001 Э4")
 		(comment 2 "Филатов А.С.")
 		(comment 3 "Сизякин А.В.")
@@
 			)
 		)
-	)
-	(text "НВЦТ.0001.0000.100"
-		(exclude_from_sim no)
-		(at 16.764 332.232 90)
-		(effects
-			(font
-				(size 2.5 2.5)
-			)
-		)

Commit message: VER1.0: исправил Э4
Other:
- note added: "ООО "Центр Водородных"
- note added: "технологий""
- note removed: "ООО "Электротранспортные"
- note removed: "технологии""

Commit message: VER1.0: исправил Э3
Parts:
- added F1, F2: Fuse, symbol Device:Fuse
Other:
- note added: "- для жгута поз.13 кабель МКЭШ 2х2,5 мм2;"
- note added: "- для жгутов поз.1-9 провод ПГУВ 1х0,5 мм2;"
- note added: "- для жгутов поз.10-11 провод ПГУВ 1х1,5 мм2;"
- note added: "- для жгутов поз.12, 14-16 кабель ПГВУЭ-35/5;"
- note added: "1 Подключение ЭХГ и датчика температуры 2 опционально."
- note added: "2 Для проводов применяемых в жгутах:"
- note added: "3 Кабели от ГРЩ обжать наконечниками ТМЛ 35-8-9."
- note added: "A3-XT1.VDC+,"
- note added: "A3-XT1.VDC-"
- note added: "A4-XT1.U,"
- note added: "A4-XT1.V,"
- note added: "A4-XT1.W"
- note added: "F1"
- note added: "F2"
- note added: "ВК1"
- note added: "Датчик температуры 2"
- note added: "ООО "Электротранспортные"
- note added: "ЭХГ"
- note added: "технологии""
- note removed: "CAN разъём"
- note removed: "А10"
- note removed: "ООО "Центр Водородных"
- note removed: "технологий""
